File: PaperCam_Kicad/PaperCam_Kicad.kicad_sch (KiCad schematic)
At the start: 11 parts, among them U1 2465

Commit message: added software
Connections:
- net DIN: now also RaspberryPiGPIO1.37, U1.6 (LBO)
- no-connect marks 34 -> 32
Changed lines of the file:
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@@
+	)
+	(junction
+		(at 34.29 88.9)
+		(diameter 0)
+		(color 0 0 0 0)
 	)
 	(junction
@@
 	)
 	(junction
+		(at 34.29 83.82)
+		(diameter 0)
+		(color 0 0 0 0)
+	)
+	(junction
 		(at 72.39 59.69)
 		(diameter 0)
@@
 	)
 	(no_connect
-		(at 43.18 80.01)
-	)
-	(no_connect
 		(at 50.8 82.55)
 	)
@@
 	)
 	(no_connect
-		(at 58.42 119.38)
-	)
-	(no_connect
 		(at 43.18 39.37)
 	)
@@
 	(wire
 		(pts
+			(xy 34.29 88.9) (xy 34.29 93.98)
+		)
+		(stroke
+			(width 0)
+			(type default)
+		)
+	)
+	(wire
+		(pts
 			(xy 128.27 40.64) (xy 128.27 90.17)
 		)
@@
 	(wire
 		(pts
+			(xy 34.29 83.82) (xy 34.29 88.9)
+		)
+		(stroke
+			(width 0)
+			(type default)
+		)
+	)
+	(wire
+		(pts
+			(xy 58.42 119.38) (xy 68.58 119.38)
+		)
+		(stroke
+			(width 0)
+			(type default)
+		)
+	)
+	(wire
+		(pts
 			(xy 77.47 64.77) (xy 92.71 64.77)
 		)
@@
 	(wire
 		(pts
+			(xy 68.58 93.98) (xy 34.29 93.98)
+		)
+		(stroke
+			(width 0)
+			(type default)
+		)
+	)
+	(wire
+		(pts
 			(xy 102.87 48.26) (xy 102.87 52.07)
 		)
@@
 	(wire
 		(pts
+			(xy 34.29 80.01) (xy 34.29 83.82)
+		)
+		(stroke
+			(width 0)
+			(type default)
+		)
+	)
+	(wire
+		(pts
 			(xy 102.87 52.07) (xy 72.39 52.07)
 		)
@@
 	(wire
 		(pts
-			(xy 34.29 83.82) (xy 34.29 88.9)
-		)
-		(stroke
-			(width 0)
-			(type default)
-		)
-	)
-	(wire
-		(pts
 			(xy 68.58 59.69) (xy 68.58 69.85)
 		)
@@
 	(wire
 		(pts
+			(xy 68.58 119.38) (xy 68.58 93.98)
+		)
+		(stroke
+			(width 0)
+			(type default)
+		)
+	)
+	(wire
+		(pts
 			(xy 27.94 119.38) (xy 27.94 143.51)
 		)
@@
 		)
 		(stroke
+			(width 0)
+			(type default)
+		)
+	)
+	(wire
+		(pts
+			(xy 34.29 80.01) (xy 43.18 80.01)
+		)
+		(stroke
