File: PaperCam_Kicad/PaperCam_Kicad.kicad_sch (KiCad schematic)
At the start: 12 parts, among them U1 2465

Commit message: fixed wiring
Connections:
- net RST: now also RaspberryPiGPIO1.11; no longer RaspberryPiGPIO1.18
- net at CameraButton1.1: now also RaspberryPiGPIO1.12; no longer RaspberryPiGPIO1.11
Other:
- moved on the sheet: CameraButton1
Changed lines of the file:
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@@
-	)
-	(no_connect
-		(at 50.8 46.99)
 	)
 	(no_connect
@@
 		(at 58.42 111.76)
 	)
+	(no_connect
+		(at 50.8 54.61)
+	)
 	(wire
 		(pts
@@
 	(wire
 		(pts
-			(xy 50.8 54.61) (xy 73.66 54.61)
-		)
-		(stroke
-			(width 0)
-			(type default)
-		)
-	)
-	(wire
-		(pts
 			(xy 29.21 29.21) (xy 34.29 29.21)
 		)
@@
 	(wire
 		(pts
+			(xy 85.09 90.17) (xy 19.05 90.17)
+		)
+		(stroke
+			(width 0)
+			(type default)
+		)
+	)
+	(wire
+		(pts
 			(xy 81.28 62.23) (xy 92.71 62.23)
 		)
@@
 	(wire
 		(pts
+			(xy 82.55 72.39) (xy 92.71 72.39)
+		)
+		(stroke
+			(width 0)
+			(type default)
+		)
+	)
+	(wire
+		(pts
 			(xy 88.9 59.69) (xy 92.71 59.69)
 		)
@@
 	(wire
 		(pts
+			(xy 85.09 90.17) (xy 85.09 80.01)
+		)
+		(stroke
+			(width 0)
+			(type default)
+		)
+	)
+	(wire
+		(pts
 			(xy 58.42 119.38) (xy 68.58 119.38)
 		)
@@
 	(wire
 		(pts
-			(xy 27.94 46.99) (xy 43.18 46.99)
+			(xy 82.55 80.01) (xy 82.55 72.39)
+		)
+		(stroke
+			(width 0)
+			(type default)
+		)
+	)
+	(wire
+		(pts
+			(xy 19.05 46.99) (xy 43.18 46.99)
 		)
 		(stroke
@@
 	(wire
 		(pts
-			(xy 73.66 72.39) (xy 92.71 72.39)
-		)
-		(stroke
-			(width 0)
-			(type default)
-		)
-	)
-	(wire
-		(pts
 			(xy 27.94 143.51) (xy 78.74 143.51)
 		)
@@
 	(wire
 		(pts
-			(xy 73.66 54.61) (xy 73.66 72.39)
+			(xy 85.09 80.01) (xy 82.55 80.01)
+		)
+		(stroke
+			(width 0)
+			(type default)
+		)
+	)
+	(wire
+		(pts
+			(xy 19.05 90.17) (xy 19.05 46.99)
+		)
+		(stroke
+			(width 0)
+			(type default)
+		)
+	)
+	(wire
+		(pts
+			(xy 64.77 48.26) (xy 50.8 48.26)
 		)
 		(stroke
@@
 		(pts
 			(xy 74.93 74.93) (xy 92.71 74.93)
+		)
+		(stroke
+			(width 0)
+			(type default)
+		)
+	)
+	(wire
+		(pts
+			(xy 50.8 48.26) (xy 50.8 46.99)
 		)
 		(stroke
@@
 	(symbol
 		(lib_id "Switch:SW_Push")
-		(at 22.86 46.99 180)
+		(at 69.85 48.26 0)
 		(unit 1)
 		(exclude_from_sim no)
@@
 		(fields_autoplaced yes)
 		(property "Reference" "CameraButton1"
-			(at 22.86 41.91 0)
+			(at 69.85 40.64 0)
 			(effects
 				(font
@@
 		)
 		(property "Value" "SW_Push"
-			(at 22.86 44.45 0)
+			(at 69.85 43.18 0)
 			(effects
 				(font
@@
 		)
 		(property "Footprint" "Button_Switch_THT:SW_PUSH-12mm"
-			(at 22.86 52.07 0)
+			(at 69.85 43.18 0)
 			(effects
 				(font
@@
 		)
 		(property "Datasheet" "~"
-			(at 22.86 52.07 0)
+			(at 69.85 43.18 0)
 			(effects
 				(font
@@
 		)
 		(property "Description" "Push button switch, generic, two pins"
-			(at 22.86 46.99 0)
+			(at 69.85 48.26 0)
 			(effects
 				(font
@@
 	)
 	(symbol
+		(lib_id "power:GND")
+		(at 74.93 48.26 90)
+		(unit 1)
+		(exclude_from_sim no)
+		(in_bom yes)
+		(on_board yes)
+		(dnp no)
+		(fields_autoplaced yes)
+		(property "Reference" "#PWR08"
+			(at 81.28 48.26 0)
+			(effects
+				(font
+					(size 1.27 1.27)
+				)
+				(hide yes)
+			)
+		)
+		(property "Value" "GND"
+			(at 78.74 48.2599 90)
+			(effects
+				(font
+					(size 1.27 1.27)
+				)
+				(justify right)
+			)
+		)
+		(property "Footprint" ""
+			(at 74.93 48.26 0)
+			(effects
+				(font
+					(size 1.27 1.27)
+				)
+				(hide yes)
+			)
+		)
+		(property "Datasheet" ""
+			(at 74.93 48.26 0)
+			(effects
+				(font
+					(size 1.27 1.27)
+				)
+				(hide yes)
+			)
+		)
+		(property "Description" "Power symbol creates a global label with name \"GND\" , ground"
+			(at 74.93 48.26 0)
+			(effects
+				(font
+					(size 1.27 1.27)
+				)
+				(hide yes)
+			)
+		)
+		(pin "1"
+		)
+		(instances
+			(project ""
+				(path "/18479ce8-91d2-4773-aac9-805b16dd781e"
+					(reference "#PWR08")
+					(unit 1)
+				)
+			)
+		)
+	)
+	(symbol
 		(lib_id "power:PWR_FLAG")
 		(at 58.42 106.68 0)
@@
 					(unit 1)
 				)
-			)
-		)
-	)
-	(symbol
-		(lib_id "power:GND")
-		(at 17.78 46.99 270)
-		(unit 1)
-		(exclude_from_sim no)
-		(in_bom yes)
-		(on_board yes)
-		(dnp no)
-		(fields_autoplaced yes)
-		(property "Reference" "#PWR08"
-			(at 11.43 46.99 0)
-			(effects
-				(font
-					(size 1.27 1.27)
-				)
-				(hide yes)
-			)
-		)
-		(property "Value" "GND"
-			(at 13.97 46.9899 90)
-			(effects
-				(font
-					(size 1.27 1.27)
-				)
-				(justify right)
-			)
-		)
-		(property "Footprint" ""
-			(at 17.78 46.99 0)
-			(effects
-				(font
-					(size 1.27 1.27)
-				)
-				(hide yes)
-			)
-		)
-		(property "Datasheet" ""
-			(at 17.78 46.99 0)
-			(effects
-				(font
-					(size 1.27 1.27)
-				)
-				(hide yes)
-			)
-		)
-		(property "Description" "Power symbol creates a global label with name \"GND\" , ground"
-			(at 17.78 46.99 0)
-			(effects
-				(font
-					(size 1.27 1.27)
-				)
-				(hide yes)
-			)
-		)
-		(pin "1"
-		)
-		(instances
-			(project ""
-				(path "/18479ce8-91d2-4773-aac9-805b16dd781e"
-					(reference "#PWR08")
-					(unit 1)
-				)

Commit message: fixed keyboard
Connections:
- net BUSY: now also RaspberryPiGPIO1.18; no longer RaspberryPiGPIO1.16
Changed lines of the file:
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@@
+	)
+	(no_connect
+		(at 50.8 52.07)
 	)
 	(no_connect
@@
 		(at 58.42 111.76)
 	)
-	(no_connect
-		(at 50.8 54.61)
-	)
 	(wire
 		(pts
@@
 	(wire
 		(pts
-			(xy 74.93 52.07) (xy 74.93 74.93)
-		)
-		(stroke
-			(width 0)
-			(type default)
-		)
-	)
-	(wire
-		(pts
 			(xy 68.58 119.38) (xy 68.58 92.71)
 		)
@@
 	(wire
 		(pts
-			(xy 50.8 52.07) (xy 74.93 52.07)
-		)
-		(stroke
-			(width 0)
-			(type default)
-		)
-	)
-	(wire
-		(pts
 			(xy 27.94 119.38) (xy 27.94 143.51)
 		)
@@
 	(wire
 		(pts
+			(xy 74.93 74.93) (xy 74.93 54.61)
+		)
+		(stroke
+			(width 0)
+			(type default)
+		)
+	)
+	(wire
+		(pts
 			(xy 36.83 62.23) (xy 36.83 87.63)
 		)
@@
 		)
 		(stroke
+			(width 0)
+			(type default)
+		)
+	)
+	(wire
+		(pts
+			(xy 50.8 54.61) (xy 74.93 54.61)
+		)
+		(stroke
