File: PaperCam_Kicad/PaperCam_Kicad.kicad_pcb (KiCad board)
At the start: 2 copper layers, 110 x 110 mm, 14 parts, among them U1 2465

Commit message: cad files
Parts:
- moved G*** 16.7 mm to (83.3, 69.1)
Connections:
- RaspberryPiGPIO1 pad 37: unconnected-(RaspberryPiGPIO1-Pad37) -> /DIN
- U1 pad 6: unconnected-(U1-LBO-Pad6) -> /DIN
Routing:
- net GND: track 0.00 -> 389.3 mm
- net +5V: track 0.00 -> 211.7 mm
- net Net-(CameraButton1-Pad1): track 0.00 -> 169.1 mm, vias 0 -> 1
- net /DIN: track 0.00 -> 149.8 mm, vias 0 -> 5
- net /BUSY: track 0.00 -> 94.1 mm, vias 0 -> 4
- net /DC: track 0.00 -> 91.4 mm, vias 0 -> 6
- net /RST: track 0.00 -> 91.3 mm, vias 0 -> 4
- net /CS: track 0.00 -> 86.1 mm, vias 0 -> 3
- net /CLK: track 0.00 -> 84.8 mm, vias 0 -> 4
- net +3V3: track 0.00 -> 84.3 mm
- net Net-(PowerSwitch1-B): track 0.00 -> 54.5 mm
