File: PaperCam_Kicad/PaperCam_Kicad.kicad_pcb (KiCad board)
At the start: 2 copper layers, 110 x 110 mm, 15 parts, among them U1 2465

Commit message: fixed wiring
Parts:
- moved G*** 23.8 mm to (83.3, 45.2)
Connections:
- RaspberryPiGPIO1 pad 11: Net-(CameraButton1-Pad1) -> /RST
- RaspberryPiGPIO1 pad 12: unconnected-(RaspberryPiGPIO1-Pad12) -> Net-(CameraButton1-Pad1)
- RaspberryPiGPIO1 pad 18: /RST -> unconnected-(RaspberryPiGPIO1-Pad18)
Routing:
- net /RST: track 98.5 -> 117.3 mm
- net Net-(CameraButton1-Pad1): track 114.0 -> 131.9 mm
Other:
- board text added: "V3!"

Commit message: fixed keyboard
Connections:
- RaspberryPiGPIO1 pad 16: /BUSY -> unconnected-(RaspberryPiGPIO1-Pad16)
- RaspberryPiGPIO1 pad 18: unconnected-(RaspberryPiGPIO1-Pad18) -> /BUSY
Routing:
- net /RST: track 117.3 -> 108.8 mm
- net /DC: track 92.8 -> 96.3 mm
- net /CS: track 91.9 -> 94.5 mm
- net /BUSY: track 100.2 -> 97.7 mm
Other:
- board text added: "V4!"
- board text removed: "V3!"
Changed lines of the file:
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@@
 	(net 24 "unconnected-(RaspberryPiGPIO1-Pad40)")
 	(net 25 "unconnected-(RaspberryPiGPIO1-Pad7)")
-	(net 26 "unconnected-(RaspberryPiGPIO1-Pad18)")
+	(net 26 "unconnected-(RaspberryPiGPIO1-Pad16)")
 	(net 27 "unconnected-(RaspberryPiGPIO1-Pad3)")
 	(net 28 "unconnected-(RaspberryPiGPIO1-Pad27)")
@@
 			(layers "*.Cu" "*.Mask")
 			(remove_unused_layers no)
-			(net 5 "/BUSY")
+			(net 26 "unconnected-(RaspberryPiGPIO1-Pad16)")
 			(pinfunction "16")
-			(pintype "passive")
+			(pintype "passive+no_connect")
 		)
 		(pad "17" thru_hole oval
@@
 			(layers "*.Cu" "*.Mask")
 			(remove_unused_layers no)
-			(net 26 "unconnected-(RaspberryPiGPIO1-Pad18)")
+			(net 5 "/BUSY")
 			(pinfunction "18")
-			(pintype "passive+no_connect")
+			(pintype "passive")
 		)
 		(pad "19" thru_hole oval
@@
 		)
 	)
-	(gr_text "V3!"
+	(gr_text "V4!"
 		(at 85.725 92.86875 0)
 		(layer "F.SilkS")
@@
 			(justify left bottom)
 		)
-		(render_cache "V3!" 0
+		(render_cache "V4!" 0
 			(polygon
 				(pts
@@
 			(polygon
 				(pts
-					(xy 92.998063 87.971694) (xy 93.172643 87.828307) (xy 93.329086 87.663156) (xy 93.460563 87.483714)
-					(xy 93.570548 87.285247) (xy 93.654238 87.076139) (xy 93.713761 86.850431) (xy 93.75375 86.436383)
-					(xy 93.740387 86.164929) (xy 93.701553 85.918663) (xy 93.640344 85.700454) (xy 93.558114 85.505477)
-					(xy 93.456655 85.333166) (xy 93.337761 85.182962) (xy 93.047316 84.941927) (xy 92.68848 84.780834)
-					(xy 92.264119 84.706702) (xy 92.142786 84.703175) (xy 91.740353 84.757198) (xy 91.547192 84.824268)
-					(xy 91.363054 84.917348) (xy 91.19138 85.035049) (xy 91.033211 85.177391) (xy 90.860083 85.3862)
-					(xy 91.489253 85.915779) (xy 91.654329 85.734332) (xy 91.897946 85.617025) (xy 92.142786 85.583243)
-					(xy 92.296612 85.596712) (xy 92.435196 85.636283) (xy 92.553768 85.698303) (xy 92.655881 85.782492)
-					(xy 92.806705 86.013376) (xy 92.879597 86.332018) (xy 92.883513 86.436383) (xy 92.831645 86.763407)
-					(xy 92.681687 87.049511) (xy 92.43994 87.283978) (xy 92.117796 87.447041) (xy 91.933665 87.4944)
-					(xy 91.740485 87.515493) (xy 91.688005 87.516486) (xy 91.688005 88.396127) (xy 91.721345 88.396127)
-					(xy 92.044911 88.448445) (xy 92.363074 88.607425) (xy 92.644351 88.868569) (xy 92.758482 89.030476)
-					(xy 92.850257 89.209661) (xy 92.914762 89.396991) (xy 92.952584 89.595951) (xy 92.961732 89.755338)
-					(xy 92.948336 89.984392) (xy 92.909275 90.19019) (xy 92.848983 90.365032) (xy 92.767971 90.515686)
-					(xy 92.672748 90.63569) (xy 92.561347 90.731387) (xy 92.439695 90.799658) (xy 92.305368 90.843232)
-					(xy 92.132955 90.861514) (xy 91.874681 90.810299) (xy 91.582388 90.643981) (xy 91.455711 90.525801)
-					(xy 91.354116 90.390093) (xy 91.352049 90.386645) (xy 90.704073 90.970507) (xy 90.826396 91.150592)
-					(xy 90.964402 91.306447) (xy 91.284532 91.54902) (xy 91.661399 91.701613) (xy 92.092693 91.760417)
-					(xy 92.132955 91.760816) (xy 92.367238 91.747164) (xy 92.591255 91.706307) (xy 92.796712 91.640954)
-					(xy 92.989215 91.550367) (xy 93.162156 91.438413) (xy 93.319848 91.302932) (xy 93.458279 91.147287)
-					(xy 93.579182 90.969239) (xy 93.680666 90.769998) (xy 93.762012 90.548817) (xy 93.822178 90.30397)
-					(xy 93.859077 90.0371) (xy 93.871292 89.755338) (xy 93.819069 89.269119) (xy 93.665131 88.810433)
-					(xy 93.4146 88.392827) (xy 93.078046 88.036536)
+					(xy 93.43019 89.54419) (xy 93.812308 89.54419) (xy 93.812308 90.502477) (xy 93.43019 90.502477)
+					(xy 93.43019 91.678751) (xy 92.471903 91.678751) (xy 92.471903 90.502477) (xy 90.413852 90.502477)
+					(xy 90.413852 90.289619) (xy 90.795838 89.54419) (xy 91.8017 89.54419) (xy 92.471903 89.54419)
+					(xy 92.471903 88.14822) (xy 91.8017 89.54419) (xy 90.795838 89.54419) (xy 93.231437 84.791224)
+					(xy 93.43019 84.791224)
 				)
 			)
 			(polygon
 				(pts
-					(xy 94.65348 89.816887) (xy 95.612194 89.816887) (xy 95.631428 84.791652) (xy 94.624415 84.791652)
+					(xy 94.694513 89.816887) (xy 95.653227 89.816887) (xy 95.672461 84.791652) (xy 94.665448 84.791652)
 				)
 			)
 			(polygon
 				(pts
-					(xy 94.65348 90.720464) (xy 94.65348 91.678751) (xy 95.612194 91.678751) (xy 95.612194 90.720464)
+					(xy 94.694513 90.720464) (xy 94.694513 91.678751) (xy 95.653227 91.678751) (xy 95.653227 90.720464)
 				)
 			)
@@
 	)
 	(segment
-		(start 103.460219 58.771438)
-		(end 103.460219 58.771437)
-		(width 0.2)
-		(layer "F.Cu")
-		(net 4)
-	)
-	(segment
-		(start 70.6355 99.6115)
-		(end 70.6355 91.596157)
+		(start 37.9345 105.95325)
+		(end 70.259249 105.95325)
 		(width 0.2)
 		(layer "F.Cu")
@@
 	)
 	(segment
-		(start 70.6355 91.596157)
-		(end 103.460219 58.771438)
+		(start 73.40738 88.824276)
+		(end 103.460219 58.771437)
 		(width 0.2)
 		(layer "F.Cu")
@@
 	)
 	(segment
-		(start 64.29375 105.95325)
-		(end 70.6355 99.6115)
+		(start 73.40738 102.805119)
+		(end 73.40738 88.824276)
 		(width 0.2)
 		(layer "F.Cu")
@@
 	)
 	(segment
-		(start 37.9345 105.95325)
-		(end 64.29375 105.95325)
+		(start 70.259249 105.95325)
+		(end 73.40738 102.805119)
 		(width 0.2)
 		(layer "F.Cu")
@@
 	)
 	(segment
+		(start 33.6565 106.75525)
+		(end 35.71875 106.75525)
+		(width 0.2)
+		(layer "F.Cu")
+		(net 5)
+	)
+	(segment
 		(start 71.8385 106.75525)
 		(end 76.2 102.39375)
@@
 	)
 	(segment
-		(start 28.64375 104.2825)
-		(end 31.1165 106.75525)
+		(start 31.18375 104.2825)
+		(end 33.6565 106.75525)
 		(width 0.2)
 		(layer "F.Cu")
@@
 	)
 	(segment
-		(start 31.1165 106.75525)
+		(start 35.71875 106.75525)
 		(end 71.8385 106.75525)
 		(width 0.2)
@@
 	)
 	(segment
-		(start 70.2345 99.212683)
-		(end 70.2345 89.457156)
+		(start 39.95475 105.4335)
+		(end 68.39775 105.4335)
 		(width 0.2)
 		(layer "F.Cu")
@@
 	)
 	(segment
-		(start 39.95475 105.4335)
-		(end 64.013683 105.4335)
+		(start 38.80375 104.2825)
+		(end 39.95475 105.4335)
 		(width 0.2)
 		(layer "F.Cu")
@@
 	)
 	(segment
-		(start 64.013683 105.4335)
-		(end 70.2345 99.212683)
+		(start 68.39775 105.4335)
+		(end 71.4375 102.39375)
 		(width 0.2)
 		(layer "F.Cu")
@@
 	(segment
 		(start 38.80375 104.2825)
-		(end 39.95475 105.4335)
+		(end 39.459314 104.2825)
 		(width 0.2)
 		(layer "F.Cu")
@@
 	)
 	(segment
-		(start 38.80375 104.2825)
-		(end 39.459314 104.2825)
+		(start 71.4375 102.39375)
+		(end 71.4375 88.254156)
 		(width 0.2)
 		(layer "F.Cu")
@@
 	)
 	(segment
-		(start 70.2345 89.457156)
+		(start 71.4375 88.254156)
 		(end 103.460219 56.231437)
 		(width 0.2)
@@
 	)
 	(segment
-		(start 82.24275 100.46855)
-		(end 82.8877 101.1135)
+		(start 71.6724 106.35425)
+		(end 75.398885 102.627765)
 		(width 0.2)
-		(layer "B.Cu")
+		(layer "F.Cu")
 		(net 43)
 	)
 	(segment
-		(start 23.56375 101.7425)
-		(end 24.8377 100.46855)
+		(start 75.398885 102.627765)
+		(end 75.398885 89.372771)
 		(width 0.2)
-		(layer "B.Cu")
+		(layer "F.Cu")
 		(net 43)
 	)
 	(segment
-		(start 97.96855 101.1135)
-		(end 100.0125 99.06955)
+		(start 24.95275 103.1315)
+		(end 31.66051 103.1315)
 		(width 0.2)
-		(layer "B.Cu")
+		(layer "F.Cu")
 		(net 43)
 	)
 	(segment
-		(start 24.8377 100.46855)
-		(end 82.24275 100.46855)
+		(start 32.33475 104.8664)
+		(end 33.8226 106.35425)
 		(width 0.2)
-		(layer "B.Cu")
+		(layer "F.Cu")
 		(net 43)
 	)
 	(segment
-		(start 100.0125 99.06955)
-		(end 100.0125 64.759156)
+		(start 32.33475 103.80574)
+		(end 32.33475 104.8664)
 		(width 0.2)
-		(layer "B.Cu")
+		(layer "F.Cu")
 		(net 43)
 	)
 	(segment
-		(start 82.8877 101.1135)
-		(end 97.96855 101.1135)
+		(start 75.398885 89.372771)
+		(end 103.460219 61.311437)
 		(width 0.2)
-		(layer "B.Cu")
+		(layer "F.Cu")
 		(net 43)
 	)
 	(segment
-		(start 100.0125 64.759156)
-		(end 103.460219 61.311437)
+		(start 33.8226 106.35425)
+		(end 71.6724 106.35425)
 		(width 0.2)
-		(layer "B.Cu")
+		(layer "F.Cu")
+		(net 43)
+	)
+	(segment
+		(start 23.56375 101.7425)
+		(end 24.95275 103.1315)
+		(width 0.2)
+		(layer "F.Cu")
+		(net 43)
+	)
+	(segment
+		(start 31.66051 103.1315)
+		(end 32.33475 103.80574)
+		(width 0.2)
+		(layer "F.Cu")
 		(net 43)
 	)
